File: custom_V1/pcb_all/ErgoDOX.sch (KiCad schematic (older format))
At the start: 97 parts, among them J1 Input, J2 OutputC, J3 OutputA, J4 Conn_01x03, J5 Conn_01x01, J6 Conn_01x01, SW0:10 SW0:3, SW0:11 SW0:2, SW0:12 SW0:1, SW0:7 SW0:6, SW0:8 SW0:5, SW0:9 SW0:4, SW1:10 SW1:3, SW1:11 SW1:2, SW1:12 SW1:1, SW1:13 SW1:0, SW1:9 SW1:4, SW2:10 SW2:3, SW2:11 SW2:2, SW2:12 SW2:1, SW2:13 SW2:0, SW2:7 SW2:6, SW2:8 SW2:5, SW2:9 SW2:4, SW3:10 SW3:3, SW3:11 SW3:2, SW3:12 SW3:1, SW3:13 SW3:0, SW3:8 SW3:5, SW3:9 SW3:4, SW4:10 SW4:3, SW4:11 SW4:2, SW4:12 SW4:1, SW4:13 SW4:0, SW4:7 SW4:6, SW4:8 SW4:5, SW4:9 SW4:4, SW5:10 SW5:3, SW5:11 SW5:2, SW5:12 SW5:1, SW5:13 SW5:0, SW5:7 SW5:6, SW5:8 SW5:5, SW5:9 SW5:4, U1 USBLC6-2SC6, U2 USBLC6-2SC6, U3 USBLC6-2SC6, U4 FE1.1s, U5 Teensy-LC, U6 74LS14

Commit message: add step of custom
Parts:
- U4: symbol Interface_USB2:FE1.1s -> ErgoDOX-rescue:FE1.1s-Interface_USB2
- U5: symbol teensy:Teensy-LC -> ErgoDOX-rescue:Teensy-LC-teensy
Changed lines of the file:
@@
 	2800 9850 3500 9850
 $Comp
-L Interface_USB2:FE1.1s U4
+L ErgoDOX-rescue:FE1.1s-Interface_USB2 U4
 U 1 1 5FF3D723
 P 10950 2250
@@
 MOSI_IN
 $Comp
-L teensy:Teensy-LC U5
+L ErgoDOX-rescue:Teensy-LC-teensy U5
 U 1 1 5FF9CC95
 P 6050 2650
