File: custom_V1/pcb_logic/ErgoDOX.kicad_pcb (KiCad board)
At the start: 2 copper layers, 141.2 x 26.1 mm, 55 parts, among them J1 Input, J10 Conn_01x01, J11 Conn_01x01, J12 Conn_01x01, J13 Conn_01x01, J14 Conn_01x01, J15 Conn_01x01, J16 Conn_01x01, J17 Conn_01x01, J18 Conn_01x01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

Commit message: add V1.1 pcb
Parts:
- added C3: 10u, Capacitor_SMD:C_1206_3216Metric, F.Cu at (70.9, 50.4)
- added C5: 1u, Capacitor_SMD:C_1206_3216Metric, F.Cu at (164.5, 40.5)
- added C6: 1u, Capacitor_SMD:C_1206_3216Metric, F.Cu at (194.8, 44.1)
- added C7: 1u, Capacitor_SMD:C_1206_3216Metric, F.Cu at (203.0, 48.2)
- C2: value 0.1u -> 10u
- moved C2 134.2 mm to (68.9, 54.5), turned to 180 degrees
- moved R5 1.92 mm to (68.9, 56.9)
- moved 12MHZ1 1.25 mm to (66.8, 50.6)
- moved U1 0.34 mm to (78.5, 42.5)
Connections:
- C2 pad 1: +5V -> VD33
- U4 pad 12: Net-(U4-Pad12) -> VD18
- U4 pad 13: Net-(U4-Pad13) -> VD33
- U4 pad 17: Net-(U4-Pad17) -> +5V
- U4 pad 21: Net-(U4-Pad21) -> VD33
- U4 pad 26: Net-(U4-Pad26) -> VD33
- U4 pad 28: Net-(U4-Pad28) -> VD18
Routing:
- net +5V: track 193.3 -> 210.1 mm
- net VD18: track 0.00 -> 15.1 mm, vias 0 -> 2
- net VD33: track 0.00 -> 14.5 mm, vias 0 -> 2
- net TEENSY_USB_D+: track 34.9 -> 30.1 mm
- net TEENSY_USB_D-: track 28.2 -> 32.8 mm
- net OUTPUTA_USB_D+: track 113.5 -> 115.8 mm
- net OUTPUTA_USB_D-: track 109.7 -> 111.1 mm
- net Net-(12MHZ1-Pad2): track 5.77 -> 7.11 mm
- net Net-(12MHZ1-Pad1): track 6.59 -> 7.66 mm
- net GND: track 35.4 -> 36.1 mm
