File: custom_V1/pcb_logic/ErgoDOX.sch (KiCad schematic (older format))
At the start: 55 parts, among them J1 Input, J10 Conn_01x01, J11 Conn_01x01, J12 Conn_01x01, J13 Conn_01x01, J14 Conn_01x01, J15 Conn_01x01, J16 Conn_01x01, J17 Conn_01x01, J18 Conn_01x01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

Commit message: add V1.1 pcb
Parts:
- added C2, C3: 10u, Capacitor_SMD:C_1206_3216Metric, symbol Device:C
- added C5, C6: 1u, Capacitor_SMD:C_1206_3216Metric, symbol Device:C
- C7: renamed from C2; value 0.1u -> 1u
Connections:
- net +5V: now also U4.17 (~XRSTJ), C5.2, C6.2
- net GND: now also C2.2, C3.2, C5.1, C6.1
- net VD18: now reaches U4.12 (VD18_O)
- net VD18: now also U4.28 (VD18), C3.1
- net VD33: now reaches U4.13 (VD33)
- net VD33: now also U4.21 (VD33_O), U4.26 (OVCJ), C2.1
- no-connect marks 23 -> 18
Other:
- moved on the sheet: C1, J18, J19
Changed lines of the file:
@@
 $EndDescr
-$Comp
-L ErgoDOX-rescue:FE1.1s-Interface_USB2 U4
-U 1 1 5FF3D723
-P 10950 2250
-F 0 "U4" H 10700 1200 50  0000 C CNN
-F 1 "FE1.1s" H 11200 1200 50  0000 C CNN
-F 2 "Package_SO:SSOP-28_3.9x9.9mm_P0.635mm" H 12000 750 50  0001 C CNN
-F 3 "" H 10950 2250 50  0001 C CNN
-	1    10950 2250
-	1    0    0    -1
-$EndComp
 $Comp
 L Power_Protection:USBLC6-2SC6 U1
@@
 L power:+5V #PWR0104
 U 1 1 602083DE
-P 14900 1000
-F 0 "#PWR0104" H 14900 850 50  0001 C CNN
-F 1 "+5V" H 14950 1200 50  0000 C CNN
-F 2 "" H 14900 1000 50  0001 C CNN
-F 3 "" H 14900 1000 50  0001 C CNN
-	1    14900 1000
+P 14900 800
+F 0 "#PWR0104" H 14900 650 50  0001 C CNN
+F 1 "+5V" H 14950 1000 50  0000 C CNN
+F 2 "" H 14900 800 50  0001 C CNN
+F 3 "" H 14900 800 50  0001 C CNN
+	1    14900 800
 	1    0    0    -1
 $EndComp
@@
 L power:+5V #PWR0110
 U 1 1 6048DEF7
-P 14950 3900
-F 0 "#PWR0110" H 14950 3750 50  0001 C CNN
-F 1 "+5V" H 15000 4100 50  0000 C CNN
-F 2 "" H 14950 3900 50  0001 C CNN
-F 3 "" H 14950 3900 50  0001 C CNN
-	1    14950 3900
+P 14950 3650
+F 0 "#PWR0110" H 14950 3500 50  0001 C CNN
+F 1 "+5V" H 15000 3850 50  0000 C CNN
+F 2 "" H 14950 3650 50  0001 C CNN
+F 3 "" H 14950 3650 50  0001 C CNN
+	1    14950 3650
 	1    0    0    -1
 $EndComp
@@
 L power:+5V #PWR0116
 U 1 1 6054AECC
-P 12200 4050
-F 0 "#PWR0116" H 12200 3900 50  0001 C CNN
-F 1 "+5V" H 12250 4250 50  0000 C CNN
-F 2 "" H 12200 4050 50  0001 C CNN
-F 3 "" H 12200 4050 50  0001 C CNN
-	1    12200 4050
+P 12150 4000
+F 0 "#PWR0116" H 12150 3850 50  0001 C CNN
+F 1 "+5V" H 12200 4200 50  0000 C CNN
+F 2 "" H 12150 4000 50  0001 C CNN
+F 3 "" H 12150 4000 50  0001 C CNN
+	1    12150 4000
 	1    0    0    -1
 $EndComp
@@
 NoConn ~ 11650 2350
 NoConn ~ 10250 1350
-NoConn ~ 10250 1850
 NoConn ~ 10250 1950
-NoConn ~ 10250 2050
-NoConn ~ 10950 1150
-NoConn ~ 11050 1150
-NoConn ~ 11150 1150
-NoConn ~ 11250 1150
 $Comp
 L Device:C C1
 U 1 1 601E032D
-P 10350 1050
-F 0 "C1" V 10098 1050 50  0000 C CNN
-F 1 "10u" V 10189 1050 50  0000 C CNN
-F 2 "Capacitor_SMD:C_1206_3216Metric" H 10388 900 50  0001 C CNN
-F 3 "~" H 10350 1050 50  0001 C CNN
-	1    10350 1050
+P 9850 950
+F 0 "C1" V 9598 950 50  0000 C CNN
+F 1 "10u" V 9689 950 50  0000 C CNN
+F 2 "Capacitor_SMD:C_1206_3216Metric" H 9888 800 50  0001 C CNN
+F 3 "~" H 9850 950 50  0001 C CNN
+	1    9850 950
 	0    1    1    0
 $EndComp
@@
 L power:GND #PWR0121
 U 1 1 60211DAC
-P 10200 1050
-F 0 "#PWR0121" H 10200 800 50  0001 C CNN
-F 1 "GND" H 10200 900 50  0000 C CNN
-F 2 "" H 10200 1050 50  0001 C CNN
-F 3 "" H 10200 1050 50  0001 C CNN
-	1    10200 1050
+P 9700 950
+F 0 "#PWR0121" H 9700 700 50  0001 C CNN
+F 1 "GND" H 9700 800 50  0000 C CNN
+F 2 "" H 9700 950 50  0001 C CNN
+F 3 "" H 9700 950 50  0001 C CNN
+	1    9700 950
 	1    0    0    -1
 $EndComp
@@
 L power:+5V #PWR0122
 U 1 1 6022A6E2
-P 10500 1050
-F 0 "#PWR0122" H 10500 900 50  0001 C CNN
-F 1 "+5V" H 10500 1200 50  0000 C CNN
-F 2 "" H 10500 1050 50  0001 C CNN
-F 3 "" H 10500 1050 50  0001 C CNN
-	1    10500 1050
+P 10000 950
+F 0 "#PWR0122" H 10000 800 50  0001 C CNN
+F 1 "+5V" H 10000 1100 50  0000 C CNN
+F 2 "" H 10000 950 50  0001 C CNN
+F 3 "" H 10000 950 50  0001 C CNN
+	1    10000 950
 	1    0    0    -1
 $EndComp
@@
 	12350 9650 15950 9650
 $Comp
-L Device:C C2
+L Device:C C7
 U 1 1 6092E169
 P 13150 8500
-F 0 "C2" V 12898 8500 50  0000 C CNN
-F 1 "0.1u" V 12989 8500 50  0000 C CNN
+F 0 "C7" V 12898 8500 50  0000 C CNN
+F 1 "1u" V 12989 8500 50  0000 C CNN
 F 2 "Capacitor_SMD:C_1206_3216Metric" H 13188 8350 50  0001 C CNN
 F 3 "~" H 13150 8500 50  0001 C CNN
@@
 L Connector_Generic:Conn_01x01 J19
 U 1 1 600EA8FD
-P 3750 7300
-F 0 "J19" H 3750 7200 50  0000 C CNN
-F 1 "Conn_01x01" H 4050 7300 50  0000 C CNN
-F 2 "Connector_PinHeader_2.54mm:PinHeader_1x01_P2.54mm_Vertical" H 3750 7300 50  0001 C CNN
-F 3 "~" H 3750 7300 50  0001 C CNN
-	1    3750 7300
+P 3750 7100
+F 0 "J19" H 3750 7000 50  0000 C CNN
+F 1 "Conn_01x01" H 4050 7100 50  0000 C CNN
+F 2 "Connector_PinHeader_2.54mm:PinHeader_1x01_P2.54mm_Vertical" H 3750 7100 50  0001 C CNN
+F 3 "~" H 3750 7100 50  0001 C CNN
+	1    3750 7100
 	-1   0    0    1
 $EndComp
@@
 L Connector_Generic:Conn_01x01 J18
 U 1 1 601789B9
-P 3750 7100
-F 0 "J18" H 3750 7000 50  0000 C CNN
-F 1 "Conn_01x01" H 4050 7100 50  0000 C CNN
-F 2 "Connector_PinHeader_2.54mm:PinHeader_1x01_P2.54mm_Vertical" H 3750 7100 50  0001 C CNN
-F 3 "~" H 3750 7100 50  0001 C CNN
-	1    3750 7100
-	-1   0    0    1
-$EndComp
-Text Label 3950 7300 0    60   ~ 0
+P 3750 7300
+F 0 "J18" H 3750 7200 50  0000 C CNN
+F 1 "Conn_01x01" H 4050 7300 50  0000 C CNN
+F 2 "Connector_PinHeader_2.54mm:PinHeader_1x01_P2.54mm_Vertical" H 3750 7300 50  0001 C CNN
+F 3 "~" H 3750 7300 50  0001 C CNN
+	1    3750 7300
+	-1   0    0    1
+$EndComp
+Text Label 3950 7100 0    60   ~ 0
 ROW4
 Text Label 3950 6900 0    60   ~ 0
@@
 Text Label 3950 6300 0    60   ~ 0
 ROW0
-Text Label 3950 7100 0    60   ~ 0
+Text Label 3950 7300 0    60   ~ 0
 ROW5
 Text Label 2000 7500 0    60   ~ 0
@@
 Text Label 2000 7100 0    60   ~ 0
 COL4
+$Comp
+L power:+5V #PWR0139
+U 1 1 6020ED87
+P 10050 1850
+F 0 "#PWR0139" H 10050 1700 50  0001 C CNN
+F 1 "+5V" H 10050 2000 50  0000 C CNN
+F 2 "" H 10050 1850 50  0001 C CNN
+F 3 "" H 10050 1850 50  0001 C CNN
+	1    10050 1850
+	1    0    0    -1
+$EndComp
+Wire Wire Line
+	10250 1850 10050 1850
+NoConn ~ 11650 2650
+$Comp
+L ErgoDOX-rescue:FE1.1s-Interface_USB2 U4
+U 1 1 5FF3D723
+P 10950 2250
+F 0 "U4" H 10700 1200 50  0000 C CNN
+F 1 "FE1.1s" H 11200 1200 50  0000 C CNN
+F 2 "Package_SO:SSOP-28_3.9x9.9mm_P0.635mm" H 12000 750 50  0001 C CNN
+F 3 "" H 10950 2250 50  0001 C CNN
+	1    10950 2250
+	1    0    0    -1
+$EndComp
+Wire Wire Line
+	10950 1150 11000 1150
+Wire Wire Line
+	11150 1150 11200 1150
+$Comp
+L Device:C C2
+U 1 1 60231BDE
+P 10650 900
+F 0 "C2" V 10398 900 50  0000 C CNN
+F 1 "10u" V 10489 900 50  0000 C CNN
+F 2 "Capacitor_SMD:C_1206_3216Metric" H 10688 750 50  0001 C CNN
+F 3 "~" H 10650 900 50  0001 C CNN
+	1    10650 900
+	0    1    1    0
+$EndComp
+$Comp
+L power:GND #PWR0140
+U 1 1 60231BE5
+P 10500 900
+F 0 "#PWR0140" H 10500 650 50  0001 C CNN
+F 1 "GND" H 10500 750 50  0000 C CNN
+F 2 "" H 10500 900 50  0001 C CNN
+F 3 "" H 10500 900 50  0001 C CNN
+	1    10500 900
+	1    0    0    -1
+$EndComp
+$Comp
+L Device:C C3
+U 1 1 6023428F
+P 11500 1000
+F 0 "C3" V 11248 1000 50  0000 C CNN
+F 1 "10u" V 11339 1000 50  0000 C CNN
+F 2 "Capacitor_SMD:C_1206_3216Metric" H 11538 850 50  0001 C CNN
+F 3 "~" H 11500 1000 50  0001 C CNN
+	1    11500 1000
+	0    -1   1    0
+$EndComp
+$Comp
+L power:GND #PWR0141
+U 1 1 60234296
+P 11650 1000
+F 0 "#PWR0141" H 11650 750 50  0001 C CNN
+F 1 "GND" H 11650 850 50  0000 C CNN
+F 2 "" H 11650 1000 50  0001 C CNN
+F 3 "" H 11650 1000 50  0001 C CNN
+	1    11650 1000
+	-1   0    0    -1
+$EndComp
+Wire Wire Line
+	10800 900  11000 900
+Wire Wire Line
+	11000 900  11000 1150
+Connection ~ 11000 1150
+Wire Wire Line
+	11000 1150 11050 1150
+Wire Wire Line
+	11200 1150 11200 1000
+Wire Wire Line
+	11200 1000 11350 1000
+Connection ~ 11200 1150
+Wire Wire Line
+	11200 1150 11250 1150
+Text GLabel 11000 900  1    50   Input ~ 0
+VD33
+Text GLabel 10250 2050 0    50   Input ~ 0
+VD33
+$Comp
+L Device:C C5
+U 1 1 6026CB2C
+P 11950 4050
+F 0 "C5" V 11698 4050 50  0000 C CNN
+F 1 "1u" V 11789 4050 50  0000 C CNN
+F 2 "Capacitor_SMD:C_1206_3216Metric" H 11988 3900 50  0001 C CNN
+F 3 "~" H 11950 4050 50  0001 C CNN
+	1    11950 4050
+	0    -1   1    0
+$EndComp
+$Comp
+L Device:C C6
+U 1 1 602702FC
+P 14700 3750
+F 0 "C6" V 14448 3750 50  0000 C CNN
+F 1 "1u" V 14539 3750 50  0000 C CNN
+F 2 "Capacitor_SMD:C_1206_3216Metric" H 14738 3600 50  0001 C CNN
+F 3 "~" H 14700 3750 50  0001 C CNN
+	1    14700 3750
+	0    -1   1    0
+$EndComp
+Wire Wire Line
+	14950 3900 14950 3750
+Wire Wire Line
+	14850 3750 14950 3750
+Connection ~ 14950 3750
+Wire Wire Line
+	14950 3750 14950 3650
+Wire Wire Line
+	14550 3750 14200 3750
+Wire Wire Line
+	14200 3750 14200 3950
+Connection ~ 14200 3950
+Wire Wire Line
+	12100 4050 12150 4050
+Wire Wire Line
+	12150 4000 12150 4050
+Connection ~ 12150 4050
+Wire Wire Line
+	12150 4050 12200 4050
+$Comp
+L power:GND #PWR0142
+U 1 1 60293573
+P 11800 4050
+F 0 "#PWR0142" H 11800 3800 50  0001 C CNN
+F 1 "GND" H 11650 4000 50  0000 C CNN
+F 2 "" H 11800 4050 50  0001 C CNN
+F 3 "" H 11800 4050 50  0001 C CNN
+	1    11800 4050
+	1    0    0    -1
+$EndComp
+Wire Wire Line
+	14900 800  14900 1000
+Text GLabel 11200 1000 1    50   Input ~ 0
+VD18
 $EndSCHEMATC
